File: teensyGNC/teensyGNC.kicad_pcb (KiCad board)
At the start: 4 copper layers, 53 x 139.5 mm, 46 parts, among them J1 ESC_1_PWM, J10 ToF_OF_SH, J11 Hall_1_PH, J12 Hall_2_PH, J13 Hall_3_PH, J14 Hall_4_PH, J2 5V_In_XH, J3 ESC_2_PWM, J4 Servo_1_PWM, J5 Servo_2_PWM, J6 7V4_In, J7 Ebyte, J8 LC29H, J9 Batt_Mon_GH, U1 E28-2G4T20SX, U2 4754, U3 AP2112K-3.3, U4 4494, U5 Teensy4.1

Commit message: Reorder
Original order on 9-9 cancelled by jlcpcb for containing blind/buried vias, added DRC rule to check, removed blind/buried vias and then reordered
Other:
- board text added: "10/9/2026 - V1.0"
- board text removed: "9/9/2026 - V1.0"
Changed lines of the file:
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@@
 		(capping no)
 		(filling no)
+		(zone_defaults)
 		(pcbplotparams
 			(layerselection 0x00000000_00000000_55555555_5755f5ff)
@@
 		)
 		(property "Value" "ToF_OF_SH"
-			(at -2.75 -7 90)
+			(at -5 -0.6 90)
 			(layer "F.SilkS")
 			(effects
@@
 		)
 	)
-	(gr_text "9/9/2026 - V1.0\n"
+	(gr_text "10/9/2026 - V1.0\n"
 		(at 98.5 58.75 0)
 		(layer "F.SilkS")
@@
 		(net "GND")
 	)
-	(via blind
+	(via
 		(at 121.75 152.25)
 		(size 0.889)
 		(drill 0.381)
-		(layers "F.Cu" "In1.Cu")
+		(layers "F.Cu" "B.Cu")
 		(free yes)
 		(net "GND")
@@
 		(net "GND")
 	)
-	(via blind
+	(via
 		(at 120.25 156.75)
 		(size 0.889)
 		(drill 0.381)
-		(layers "F.Cu" "In1.Cu")
+		(layers "F.Cu" "B.Cu")
 		(free yes)
 		(net "GND")
@@
 		(net "GND")
 	)
-	(via blind
+	(via
 		(at 111 152.25)
 		(size 0.889)
 		(drill 0.381)
-		(layers "F.Cu" "In1.Cu")
+		(layers "F.Cu" "B.Cu")
 		(free yes)
 		(net "GND")
 	)
-	(via blind
+	(via
 		(at 109.25 156.75)
 		(size 0.889)
 		(drill 0.381)
-		(layers "F.Cu" "In1.Cu")
+		(layers "F.Cu" "B.Cu")
 		(free yes)
 		(net "GND")
@@
 		(net "GND")
 	)
-	(via blind
+	(via
 		(at 107.75 142.25)
 		(size 0.889)
 		(drill 0.381)
-		(layers "F.Cu" "In1.Cu")
+		(layers "F.Cu" "B.Cu")
 		(free yes)
 		(net "GND")
@@
 		(net "GND")
 	)
-	(via blind
+	(via
 		(at 107.75 145.25)
 		(size 0.889)
 		(drill 0.381)
-		(layers "F.Cu" "In1.Cu")
+		(layers "F.Cu" "B.Cu")
 		(free yes)
 		(net "GND")
@@
 		(net "GND")
 	)
-	(via blind
+	(via
 		(at 110.875 149.375)
 		(size 0.889)
 		(drill 0.381)
-		(layers "F.Cu" "In1.Cu")
+		(layers "F.Cu" "B.Cu")
 		(free yes)
 		(net "GND")
@@
 		(net "GND")
 	)
-	(via blind
+	(via
 		(at 108.05 140.95)
 		(size 0.889)
 		(drill 0.381)
-		(layers "F.Cu" "In1.Cu")
+		(layers "F.Cu" "B.Cu")
 		(free yes)
 		(net "GND")
@@
 		(net "GND")
 	)
-	(via blind
+	(via
 		(at 121.75 149.25)
 		(size 0.889)
 		(drill 0.381)
-		(layers "F.Cu" "In1.Cu")
+		(layers "F.Cu" "B.Cu")
 		(free yes)
 		(net "GND")
@@
 		(net "GND")
 	)
-	(via blind
+	(via
 		(at 108.05 135.45)
 		(size 0.889)
 		(drill 0.381)
-		(layers "F.Cu" "In1.Cu")
+		(layers "F.Cu" "B.Cu")
 		(free yes)
 		(net "GND")

Commit message: ! CRITICAL FIX !
5V Input plug was placed the wrong way around, now flipped back to the correct direction on the board. For the V1.0 deliveries, the first board might have had its ebyte power voltage converter fried (not tested yet), jst xh flipped manually (steps in notebook) for successful testing of altitude control on vehicle. For second board, will need to flip the jst xh first.
Parts:
- turned J2 to 0 degrees
Connections:
- J2 pad 1: +5V -> GND
- J2 pad 2: GND -> +5V
Changed lines of the file:
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@@
 		(capping no)
 		(filling no)
-		(zone_defaults)
 		(pcbplotparams
 			(layerselection 0x00000000_00000000_55555555_5755f5ff)
@@
 	(footprint "Connector_JST:JST_XH_B2B-XH-AM_1x02_P2.50mm_Vertical"
 		(layer "F.Cu")
-		(at 98.6 52 180)
+		(at 98.6 52)
 		(descr "JST XH series connector, B2B-XH-AM, with boss (http://www.jst-mfg.com/product/pdf/eng/eXH.pdf)")
 		(tags "connector JST XH vertical boss")
@@
 		)
 		(property "LCSC Part #" "C158012"
-			(at -1.25 0 180)
+			(at -1.25 0 0)
 			(unlocked yes)
 			(layer "F.Fab")
@@
 		)
 		(property "LCSC Part" ""
-			(at -1.25 0 180)
+			(at -1.25 0 0)
 			(unlocked yes)
 			(layer "F.Fab")
@@
 		(duplicate_pad_numbers_are_jumpers no)
 		(fp_line
-			(start 3.8 -0.2)
-			(end 3.05 -0.2)
+			(start -4.1 -2.75)
+			(end -4.1 -1.5)
 			(stroke
 				(width 0.12)
@@
 		)
 		(fp_line
-			(start 3.05 2.75)
-			(end 0 2.75)
+			(start -3.8 -0.2)
+			(end -3.05 -0.2)
 			(stroke
 				(width 0.12)
@@
 		)
 		(fp_line
-			(start 3.05 -0.2)
-			(end 3.05 2.75)
+			(start -3.05 -0.2)
+			(end -3.05 1.14)
 			(stroke
 				(width 0.12)
@@
 		)
 		(fp_line
-			(start 0 2.75)
-			(end -1.99 2.75)
+			(start -2.85 -2.75)
+			(end -4.1 -2.75)
 			(stroke
 				(width 0.12)
@@
 		)
 		(fp_line
-			(start -2.85 -2.75)
-			(end -4.1 -2.75)
+			(start 0 2.75)
+			(end -1.99 2.75)
 			(stroke
 				(width 0.12)
@@
 		)
 		(fp_line
-			(start -3.05 -0.2)
-			(end -3.05 1.14)
+			(start 3.05 -0.2)
+			(end 3.05 2.75)
 			(stroke
 				(width 0.12)
@@
 		)
 		(fp_line
-			(start -3.8 -0.2)
-			(end -3.05 -0.2)
+			(start 3.05 2.75)
+			(end 0 2.75)
 			(stroke
 				(width 0.12)
@@
 		)
 		(fp_line
-			(start -4.1 -2.75)
-			(end -4.1 -1.5)
+			(start 3.8 -0.2)
+			(end 3.05 -0.2)
 			(stroke
 				(width 0.12)
@@
 		)
 		(fp_rect
-			(start 2 -2.45)
-			(end 3.8 -1.7)
+			(start -3.81 -2.46)
+			(end 3.81 3.51)
 			(stroke
 				(width 0.12)
@@
 		)
 		(fp_rect
-			(start -0.5 -2.45)
-			(end 0.5 -1.7)
+			(start -3.8 -2.45)
+			(end -2 -1.7)
 			(stroke
 				(width 0.12)
@@
 		)
 		(fp_rect
-			(start -3.8 -2.45)
-			(end -2 -1.7)
+			(start -0.5 -2.45)
+			(end 0.5 -1.7)
 			(stroke
 				(width 0.12)
@@
 		)
 		(fp_rect
-			(start -3.81 -2.46)
-			(end 3.81 3.51)
+			(start 2 -2.45)
+			(end 3.8 -1.7)
 			(stroke
 				(width 0.12)
@@
 		)
 		(fp_line
-			(start -1.25 -1.35)
-			(end -0.625 -2.35)
+			(start -1.875 -2.35)
+			(end -1.25 -1.35)
 			(stroke
 				(width 0.1)
@@
 		)
 		(fp_line
-			(start -1.875 -2.35)
-			(end -1.25 -1.35)
+			(start -1.25 -1.35)
+			(end -0.625 -2.35)
 			(stroke
 				(width 0.1)
@@
 		)
 		(pad "1" thru_hole roundrect
-			(at -1.25 0 180)
+			(at -1.25 0)
 			(size 1.7 2)
 			(drill 1)
@@
 			(remove_unused_layers no)
 			(roundrect_rratio 0.147059)
-			(net "+5V")
+			(net "GND")
 			(pinfunction "Pin_1_1")
 			(pintype "passive")
 		)
 		(pad "2" thru_hole oval
-			(at 1.25 0 180)
+			(at 1.25 0)
 			(size 1.7 2)
 			(drill 1)
 			(layers "*.Cu" "*.Mask")
 			(remove_unused_layers no)
-			(net "GND")
+			(net "+5V")
 			(pinfunction "Pin_2_2")
 			(pintype "passive")
